File: Ingalls_KiCad.kicad_sch (KiCad schematic)
At the start: 83 parts, among them IC1 NJM2845DL1-05-TE1, IC2 A3982SLBTR-T, IC3 NJM2845DL1-33-TE1, IC4 TD62083AF, IC5 A3982SLBTR-T, J1 B4B-XH-A, J2 MOTOR_CON_R, J3 MOTOR_CON_L, J4 Conn_01x04_Socket, J5 B4B-XH-A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

Commit message: Footprint data changed
Parts:
- F1: footprint RUSBF1102 -> LIB_RUSBF110-2:RUSBF1102
- IC1: footprint TO-252-3-L1 -> LIB_NJM2845DL1-05-TE1:TO-252-3-L1
- IC2, IC5: footprint A3959SLBTRT -> A3982SLBTR-T:A3959SLBTRT
- IC3: footprint NJM2845DL133TE1 -> LIB_NJM2845DL1-33-TE1:NJM2845DL133TE1
- IC4: footprint SOIC127P1030X245-18N -> LIB_TD62083AF:SOIC127P1030X245-18N
- J1, J5: footprint B4BXHA -> B4B-XH-A:B4BXHA
- LED_IR_LF1, LED_IR_LS1, LED_IR_RF1, LED_IR_RS1: footprint SFH4545 -> LIB_SFH_4545:SFH4545
- LS1: footprint PKM13EPYH4000A0 -> PKM13EPYH4000-A0:PKM13EPYH4000A0
- PT_LF1, PT_LF2, PT_LF3, PT_LF4: footprint TEFT4300 -> LIB_TEFT4300:TEFT4300
- Q1: footprint TJ8S06M3LT6L1NQ -> LIB_TJ8S06M3L_T6L1,NQ_:TJ8S06M3LT6L1NQ
- S1, S2, S3: footprint PTS636SL43LFS -> PTS636_SL43_LFS:PTS636SL43LFS
Changed lines of the file:
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@@
 			)
 		)
-		(property "Footprint" "TEFT4300"
+		(property "Footprint" "LIB_TEFT4300:TEFT4300"
 			(at 292.1 183.82 0)
 			(effects
@@
 			)
 		)
-		(property "Footprint" "NJM2845DL133TE1"
+		(property "Footprint" "LIB_NJM2845DL1-33-TE1:NJM2845DL133TE1"
 			(at 166.37 133.02 0)
 			(effects
@@
 			)
 		)
-		(property "Footprint" "RUSBF1102"
+		(property "Footprint" "LIB_RUSBF110-2:RUSBF1102"
 			(at 64.77 127.94 0)
 			(effects
@@
 			)
 		)
-		(property "Footprint" "TO-252-3-L1"
+		(property "Footprint" "LIB_NJM2845DL1-05-TE1:TO-252-3-L1"
 			(at 113.03 136.83 0)
 			(effects
@@
 			)
 		)
-		(property "Footprint" "SFH4545"
+		(property "Footprint" "LIB_SFH_4545:SFH4545"
 			(at 412.42 33.02 0)
 			(effects
@@
 			)
 		)
-		(property "Footprint" "PTS636SL43LFS"
+		(property "Footprint" "PTS636_SL43_LFS:PTS636SL43LFS"
 			(at 92.71 205.41 0)
 			(effects
@@
 			)
 		)
-		(property "Footprint" "B4BXHA"
+		(property "Footprint" "B4B-XH-A:B4BXHA"
 			(at 291.77 265.43 0)
 			(effects
@@
 			)
 		)
-		(property "Footprint" "SFH4545"
+		(property "Footprint" "LIB_SFH_4545:SFH4545"
 			(at 387.02 33.02 0)
 			(effects
@@
 			)
 		)
-		(property "Footprint" "PTS636SL43LFS"
+		(property "Footprint" "PTS636_SL43_LFS:PTS636SL43LFS"
 			(at 92.71 174.93 0)
 			(effects
@@
 			)
 		)
-		(property "Footprint" "SOIC127P1030X245-18N"
+		(property "Footprint" "LIB_TD62083AF:SOIC127P1030X245-18N"
 			(at 241.3 168.58 0)
 			(effects
@@
 			)
 		)
-		(property "Footprint" "PKM13EPYH4000A0"
+		(property "Footprint" "PKM13EPYH4000-A0:PKM13EPYH4000A0"
 			(at 58.42 253.67 0)
 			(effects
@@
 			)
 		)
-		(property "Footprint" "A3959SLBTRT"
+		(property "Footprint" "A3982SLBTR-T:A3959SLBTRT"
 			(at 189.23 137.49 0)
 			(effects
@@
 			)
 		)
-		(property "Footprint" "TJ8S06M3LT6L1NQ"
+		(property "Footprint" "LIB_TJ8S06M3L_T6L1,NQ_:TJ8S06M3LT6L1NQ"
 			(at 141.91 27.94 0)
 			(effects
@@
 			)
 		)
-		(property "Footprint" "PTS636SL43LFS"
+		(property "Footprint" "PTS636_SL43_LFS:PTS636SL43LFS"
 			(at 92.71 190.17 0)
 			(effects
@@
 			)
 		)
-		(property "Footprint" "B4BXHA"
+		(property "Footprint" "B4B-XH-A:B4BXHA"
 			(at 169.85 265.43 0)
 			(effects
@@
 			)
 		)
-		(property "Footprint" "SFH4545"
+		(property "Footprint" "LIB_SFH_4545:SFH4545"
 			(at 209.88 33.02 0)
 			(effects
@@
 			)
 		)
-		(property "Footprint" "SFH4545"
+		(property "Footprint" "LIB_SFH_4545:SFH4545"
 			(at 235.28 33.02 0)
 			(effects
@@
 			)
 		)
-		(property "Footprint" "A3959SLBTRT"
+		(property "Footprint" "A3982SLBTR-T:A3959SLBTRT"
 			(at 66.04 138.76 0)
 			(effects
@@
 			)
 		)
-		(property "Footprint" "TEFT4300"
+		(property "Footprint" "LIB_TEFT4300:TEFT4300"
 			(at 308.61 183.82 0)
 			(effects
@@
 			)
 		)
-		(property "Footprint" "TEFT4300"
+		(property "Footprint" "LIB_TEFT4300:TEFT4300"
 			(at 341.63 183.82 0)
 			(effects
@@
 			)
 		)
-		(property "Footprint" "TEFT4300"
+		(property "Footprint" "LIB_TEFT4300:TEFT4300"
 			(at 325.12 183.82 0)
 			(effects
