File: Ingalls_KiCad.kicad_sch (KiCad schematic)
At the start: 83 parts, among them IC1 NJM2845DL1-05-TE1, IC2 A3982SLBTR-T, IC3 NJM2845DL1-33-TE1, IC4 TD62083AF, IC5 A3982SLBTR-T, J1 B4B-XH-A, J2 MOTOR_CON_R, J3 MOTOR_CON_L, J4 Conn_01x04_Socket, J5 B4B-XH-A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

Commit message: Title added
Other:
- title: (none) -> Ingalls
Changed lines of the file:
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@@
 	(generator_version "9.0")
 	(paper "A3")
+	(title_block
+		(title "Ingalls")
+	)
 	(rectangle
 		(start 29.21 76.2)

Commit message: Changes
Parts:
- removed IC4: TD62083AF, LIB_TD62083AF:SOIC127P1030X245-18N, symbol TD62083AF:TD62083AF
- removed Q1: TJ8S06M3L_T6L1,NQ_, LIB_TJ8S06M3L_T6L1,NQ_:TJ8S06M3LT6L1NQ, symbol TJ8S06M3L_T6L1_NQ_:TJ8S06M3L_T6L1,NQ_
- removed R17, R18, R19, R20: 1k, Resistor_SMD:R_0603_1608Metric, symbol Device:R_US
- added Q2, Q3, Q4, Q5, Q6, Q7, Q8, Q9: AO3400A, SOT95P280X125-3N, symbol AO3400A:AO3400A
- C11, C5: value 0.1u -> 0.33u
- C12, C6: value 10u -> 2.2u
- R7: value 10k -> 30k
- R8: value 1k -> 10k
Connections:
- net VDD is gone; now on net 5V: J6.1 (Pin_1)
- net +5V: now also J8.21 (Pin_21)
- net GND: now also J8.22 (Pin_22), J9.1 (Pin_1), J9.21 (Pin_21), J9.22 (Pin_22), Q2.2 (S), Q3.2 (S), Q4.2 (S), Q5.2 (S), Q6.2 (S), Q7.2 (S), Q8.2 (S), Q9.2 (S)
- net LED1: now also Q6.1 (G)
- net LED2: now also Q7.1 (G)
- net LED3: now also Q8.1 (G)
- net LED4: now also Q9.1 (G)
- net SEN_LED_LF: now also Q2.1 (G)
- net SEN_LED_LS: now also Q3.1 (G)
- net SEN_LED_RF: now also Q5.1 (G)
- net SEN_LED_RS: now also Q4.1 (G)
- net at R25.2: now also Q4.3 (D)
- net at LED1.1 (K): now also Q6.3 (D)
- net at F1.1: now also SW1.1 (A)
- net at LED4.1 (K): now also Q9.3 (D)
- net at R23.2: now also Q3.3 (D)
- net at LED2.1 (K): now also Q7.3 (D)
- net at R27.2: now also Q5.3 (D)
- net at R22.2: now also Q2.3 (D)
- net at LED3.1 (K): now also Q8.3 (D)
- no-connect marks 53 -> 47
Other:
- moved on the sheet: C11, C12, C5, C6, ESP32-S3-DevKitC-1, F1, IC1, IC3, J4, LED1, LED2, LED3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

Commit message: Changes added
Parts:
- removed R10, R14, R5: 10k, Resistor_SMD:R_0603_1608Metric, symbol Device:R_US
- C4: value 1u -> 0.22u
- R13, R4: value 10k -> 20k
- R6, R9: value 0.56 -> 0.5
Connections:
- net +12V: no longer IC2.12 (MS1), IC2.13 (RESET), IC2.14 (ROSC), IC2.15 (VDD)
- net GND: now also R13.2, R4.2
- net at IC2.17 (REF), R3.2, R4.1: now also IC2.12 (MS1), IC2.13 (RESET), IC2.14 (ROSC), IC2.15 (VDD)
Other:
- note added: "4V"
- moved on the sheet: C1, C2, R3

Commit message: Changes made
Parts:
- added C19: 0.1u, Capacitor_SMD:C_0603_1608Metric, symbol Device:C
- added R10, R14, R17, R5: 100, Resistor_SMD:R_0603_1608Metric, symbol Device:R_US
Connections:
- net +3V3: now also IC2.15 (VDD), C19.1
- net GND: now also C19.2
- net at Q6.3 (D): now also R5.2; no longer LED1.1 (K)
- net at Q7.3 (D): now also R10.2; no longer LED2.1 (K)
- net at IC2.12 (MS1), IC2.14 (ROSC), IC2.17 (REF)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: no longer IC2.13 (RESET), IC2.15 (VDD)
- net at LED4.1 (K): now also R17.1; no longer Q9.3 (D)
- net at Q8.3 (D): now also R14.2; no longer LED3.1 (K)
- net RESET: now reaches ESP32-S3-DevKitC-1.8 (GPIO8)
- net RESET: now also IC2.13 (RESET)
- new net: LED1.1 (K), R5.1
- new net: LED2.1 (K), R10.1
- new net: Q9.3 (D), R17.2
- new net: LED3.1 (K), R14.1
- no-connect marks 47 -> 46
Other:
- moved on the sheet: C2, Q6, Q7, Q8, Q9, R4
