File: Ingalls_KiCad.kicad_pcb (KiCad board)
At the start: 2 copper layers, 80 x 106 mm, 80 parts, among them IC1 NJM2845DL1-05-TE1, IC2 A3982SLBTR-T, IC3 NJM2845DL1-33-TE1, IC4 TD62083AF, IC5 A3982SLBTR-T, J1 B4B-XH-A, J4 Conn_01x04_Socket, J5 B4B-XH-A, J6 Conn_01x01_Socket, J7 Conn_01x01_Socket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

Commit message: PCB updated
Parts:
- moved C12 93.8 mm to (134.1, 56.6)
- moved R8 75.4 mm to (142.4, 66.6)
- moved C15 41.8 mm to (126.6, 121.1)
- moved C8 40.5 mm to (186.9, 129.1), turned to 180 degrees
- moved C5 39.4 mm to (144.6, 121.1)
- moved IC1 36.8 mm to (114.6, 117.6), turned to 90 degrees
- moved SW1 35.5 mm to (150.8, 138.1), turned to 90 degrees
- moved C10 34.3 mm to (177.4, 122.8), turned to 90 degrees
- moved Q1 34.2 mm to (154.1, 123.1)
- moved C9 32.5 mm to (180.1, 121.1), turned to 180 degrees
- moved C11 31.1 mm to (144.6, 124.1)
- moved F1 30.7 mm to (156.4, 139.3)
- moved C16 30.3 mm to (184.4, 117.1)
- moved R27 27.6 mm to (171.1, 54.6)
- moved J6 25.6 mm to (163.4, 63.6)
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Routing:
- net +5V: track 118.6 -> 0.00 mm
- net GND: track 0.00 -> 71.9 mm, vias 1 -> 15
- net +3V3: track 23.9 -> 0.00 mm
- net Net-(IC4-O6): track 0.00 -> 22.8 mm
- net Net-(IC4-O4): track 0.00 -> 20.3 mm
- net Net-(IC4-O3): track 0.00 -> 17.4 mm
- net Net-(Q1-D): track 0.00 -> 17.1 mm
- net Net-(IC4-O2): track 0.00 -> 16.7 mm
- net Net-(IC4-O5): track 15.4 -> 0.00 mm
- net Net-(IC4-O1): track 0.00 -> 13.8 mm
- net Net-(IC2-OUT1B): track 0.00 -> 12.8 mm
- net Net-(LED_IR_LF1-K): track 0.00 -> 11.8 mm
- net Net-(IC2-REF): track 0.00 -> 10.3 mm
- net Net-(BT1-+): track 0.00 -> 10.1 mm
- net Net-(LED1-K): track 0.00 -> 9.72 mm
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- added copper zone on In1.Cu, net GND
Other:
- copper layers 2 -> 4

Commit message: PCB updated
Parts:
- moved R10 2.17 mm to (144.6, 55.6), turned to 180 degrees
- moved R23 2.06 mm to (137.6, 53.6), turned to 180 degrees
- moved R9 1.50 mm to (116.4, 125.1)
- moved R28 1.36 mm to (174.9, 50.4)
- moved C12 0.71 mm to (133.6, 56.1), turned to 180 degrees
- moved J4 0.50 mm to (181.4, 67.9)
Routing:
- net MOTOR_EN: track 0.00 -> 142.2 mm, vias 0 -> 4
- net +12V: track 0.00 -> 111.6 mm, vias 0 -> 12
- net STEP_R: track 0.00 -> 95.3 mm, vias 0 -> 2
- net DIR_R: track 0.00 -> 94.9 mm, vias 0 -> 2
- net STEP_L: track 0.00 -> 84.7 mm, vias 0 -> 2
- net DIR_L: track 0.00 -> 84.0 mm, vias 0 -> 2
- net AD_LF: track 7.40 -> 77.7 mm, vias 0 -> 3
- net AD_LS: track 8.87 -> 73.1 mm, vias 0 -> 3
- net Net-(IC4-O8): track 0.00 -> 61.8 mm, vias 0 -> 2
- net BATTERY: track 0.00 -> 60.5 mm
- net Net-(IC4-O7): track 0.00 -> 55.0 mm, vias 0 -> 2
- net Net-(IC4-O5): track 0.00 -> 48.2 mm, vias 0 -> 4
- net UP: track 0.00 -> 45.3 mm, vias 0 -> 2
- net EXECUTE: track 0.00 -> 44.4 mm, vias 0 -> 2
- net AD_RF: track 0.00 -> 42.9 mm, vias 0 -> 1
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- added copper zone on In2.Cu, net +12V

Commit message: Changes made
Parts:
- removed IC4: TD62083AF, LIB_TD62083AF:SOIC127P1030X245-18N
- removed Q1: TJ8S06M3L_T6L1,NQ_, LIB_TJ8S06M3L_T6L1,NQ_:TJ8S06M3LT6L1NQ
- removed R10, R14, R5: 10k, Resistor_SMD:R_0603_1608Metric
- removed R17, R18, R19, R20: 1k, Resistor_SMD:R_0603_1608Metric
- removed SW_MODE1: ~, EG1218:SW_1218_EWI
- added Q2: AO3400A, KiCad:SOT95P280X125-3N, F.Cu at (82.4, 66.8)
- added Q3: AO3400A, KiCad:SOT95P280X125-3N, F.Cu at (82.4, 71.5)
- added Q4: AO3400A, KiCad:SOT95P280X125-3N, F.Cu at (82.4, 76.1)
- added Q5: AO3400A, KiCad:SOT95P280X125-3N, F.Cu at (82.4, 80.8)
- added Q6: AO3400A, KiCad:SOT95P280X125-3N, F.Cu at (82.4, 85.4)
- added Q7: AO3400A, KiCad:SOT95P280X125-3N, F.Cu at (87.7, 66.8)
- added Q8: AO3400A, KiCad:SOT95P280X125-3N, F.Cu at (87.7, 71.5)
- added Q9: AO3400A, KiCad:SOT95P280X125-3N, F.Cu at (87.7, 76.1)
- C11, C5: value 0.1u -> 0.33u
- C12, C6: value 10u -> 2.2u
- C4: value 1u -> 0.22u
- R13, R4: value 10k -> 20k
- R6, R9: value 0.56 -> 0.5
- R7: value 10k -> 30k
- R8: value 1k -> 10k
Connections:
- F1 pad 1: Net-(Q1-S) -> Net-(SW1-A)
- IC2 pad 12: +12V -> Net-(IC2-MS1)
- IC2 pad 13: +12V -> Net-(IC2-MS1)
- IC2 pad 14: +12V -> Net-(IC2-MS1)
- IC2 pad 15: +12V -> Net-(IC2-MS1)
- IC2 pad 17: Net-(IC2-REF) -> Net-(IC2-MS1)
- J6 pad 1: VDD -> 5V
- J8 pad 21: unconnected-(J8-Pin_21-Pad21) -> +5V
- J8 pad 22: unconnected-(J8-Pin_22-Pad22) -> GND
- J9 pad 1: unconnected-(J9-Pin_1-Pad1) -> GND
- J9 pad 21: unconnected-(J9-Pin_21-Pad21) -> GND
- J9 pad 22: unconnected-(J9-Pin_22-Pad22) -> GND
- R13 pad 2: Net-(R13-Pad2) -> GND
- R3 pad 2: Net-(IC2-REF) -> Net-(IC2-MS1)
- R4 pad 1: Net-(IC2-REF) -> Net-(IC2-MS1)
- R4 pad 2: Net-(R4-Pad2) -> GND
- SW1 pad 1: Net-(Q1-D) -> Net-(SW1-A)
Routing:
- net (no net): track 0.00 -> 68.2 mm
- net Net-(IC2-MS1): track 0.00 -> 26.5 mm
- net Net-(SW1-A): track 0.00 -> 25.8 mm
- net Net-(IC4-O4): track 20.3 -> 0.00 mm
- net Net-(IC4-O3): track 17.4 -> 0.00 mm
- net Net-(Q1-D): track 17.1 -> 0.00 mm
- net Net-(IC4-O2): track 16.7 -> 0.00 mm
- net +12V: track 111.6 -> 95.4 mm
- net Net-(IC4-O1): track 13.8 -> 0.00 mm
- net Net-(IC2-REF): track 10.3 -> 0.00 mm
- net Net-(Q1-S): track 8.71 -> 0.00 mm
- net GND: track 113.5 -> 119.0 mm
- net Net-(R13-Pad2): track 3.56 -> 0.00 mm
- net Net-(R4-Pad2): track 1.95 -> 0.00 mm
